Commit message: Set the hardware with launch arguments
use_dummy, usb_port and baud_rate were fixed in stepit.ros2_control.xacro,
so a robot could only be configured by editing the module. They are now
xacro arguments of stepit.urdf.xacro, which robot.launch.py sets from launch
arguments of the same names, with the values of before as defaults: StepIt
Macro sets them from its own configuration.

Co-Authored-By: Claude Opus 5.5 <noreply@anthropic.com>

File: src/robot_description/urdf/stepit.ros2_control.xacro (robot description, xacro)
@@ -1,11 +1,11 @@
 <?xml version="1.0"?>
 <robot xmlns:xacro="http://www.ros.org/wiki/xacro">
-  <xacro:macro name="stepit_ros2_control" params="name">
+  <xacro:macro name="stepit_ros2_control" params="name use_dummy:=true usb_port:=/dev/ttyACM0 baud_rate:=9600">
     <ros2_control name="${name}" type="system">
       <hardware>
         <plugin>stepit_driver/StepitHardware</plugin>
-        <param name="use_dummy">true</param>
-        <param name="usb_port">/dev/ttyACM0</param>
-        <param name="baud_rate">9600</param>
+        <param name="use_dummy">${use_dummy}</param>
+        <param name="usb_port">${usb_port}</param>
+        <param name="baud_rate">${baud_rate}</param>
         <param name="timeout">0.2</param>
       </hardware>

File: src/robot_description/urdf/stepit.urdf.xacro (robot description, xacro)
@@ -4,4 +4,12 @@
   <xacro:include filename="$(find robot_description)/urdf/stepit.ros2_control.xacro" />
   <xacro:stepit_sample_robot />
-  <xacro:stepit_ros2_control name="stepit_ros2_control" />
+  <!-- The hardware, set by the launch arguments of the same names: the fake
+       motors by default. -->
+  <xacro:arg name="use_dummy" default="true" />
+  <xacro:arg name="usb_port" default="/dev/ttyACM0" />
+  <xacro:arg name="baud_rate" default="9600" />
+  <xacro:stepit_ros2_control name="stepit_ros2_control"
+                             use_dummy="$(arg use_dummy)"
+                             usb_port="$(arg usb_port)"
+                             baud_rate="$(arg baud_rate)" />
 </robot>
